Commit message: Add: Velodyne VLP 16 Lidar

File: src/atvurdf/urdf/atvurdf_nav.urdf (robot description, URDF)
Before this commit: robot atvurdf, 2 links, 1 joints
Links:
- added link lidar_link, mass 0.125; collision cylinder length=0.0 radius=0.0; visual cylinder length=0.0 radius=0.0
- added link velodyne_vlp16, mass 0.125; collision cylinder length=0.75 radius=0.0508; visual mesh filename=file://$(find atvurdf)/meshes/VLP16_base_1.dae scale=1 1 1
Joints:
- added joint lidar_joint: type fixed, parent base_link, child lidar_link, origin xyz=0.215 0.0 0.30 rpy=0 0 0
- added joint velodyne_vlp16_joint: type fixed, parent base_link, child velodyne_vlp16, origin xyz=0.215 1.0 0.70 rpy=0 0 0

Commit message: Fix: Lidar placement and range

File: src/atvurdf/urdf/atvurdf_nav.urdf (robot description, URDF)
Before this commit: robot atvurdf, 4 links, 3 joints
Joints:
- joint velodyne_vlp16_joint: origin xyz=0.215 1.0 0.70 rpy=0 0 0 -> xyz=0.0 0.0 0.0 rpy=0 0 0
