Commit message: Add: fixed joint states and tf

File: src/atvurdf/urdf/atvurdf_skid_steer.urdf (robot description, URDF)
Before this commit: robot atvurdf, 4 links, 3 joints
Joints:
- joint base_joint: child base_footprint -> base_link; parent base_link -> base_footprint

Commit message: Frame fix

File: src/atvurdf/urdf/atvurdf_skid_steer.urdf (robot description, URDF)
Before this commit: robot atvurdf, 4 links, 3 joints
Joints:
- joint base_joint: child base_link -> base_footprint; parent base_footprint -> base_link

Commit message: Add: IMU

File: src/atvurdf/urdf/atvurdf_skid_steer.urdf (robot description, URDF)
Before this commit: robot atvurdf, 4 links, 3 joints
Links:
- added link imu_link, mass 0.125; collision cylinder length=0.0 radius=0.0; visual cylinder length=0.0 radius=0.0
Joints:
- added joint imu_joint: type fixed, parent base_link, child imu_link, origin xyz=0.0 0.0 0.0 rpy=0 0 0

Commit message: Add: measurement script, laser fix, frame fixes

File: src/atvurdf/urdf/atvurdf_skid_steer.urdf (robot description, URDF)
Before this commit: robot atvurdf, 5 links, 4 joints
Links:
- added link drivewhl_b_l_link, mass 10; collision mesh filename=file://$(find atvurdf)/meshes/rigid_left_front_wheel.stl scale=0.001 0.001 0.001; visual mesh filename=file://$(find atvurdf)/meshes/rigid_left_front_wheel.stl scale=0.001 0.001 0.001
- added link drivewhl_b_r_link, mass 10; collision mesh filename=file://$(find atvurdf)/meshes/rigid_right_front_wheels.stl scale=0.001 0.001 0.001; visual mesh filename=file://$(find atvurdf)/meshes/rigid_right_front_wheels.stl scale=0.001 0.001 0.001
- added link drivewhl_f_l_link, mass 10; collision mesh filename=file://$(find atvurdf)/meshes/rigid_left_front_wheel.stl scale=0.001 0.001 0.001; visual mesh filename=file://$(find atvurdf)/meshes/rigid_left_front_wheel.stl scale=0.001 0.001 0.001
- added link drivewhl_f_r_link, mass 10; collision mesh filename=file://$(find atvurdf)/meshes/rigid_right_front_wheels.stl scale=0.001 0.001 0.001; visual mesh filename=file://$(find atvurdf)/meshes/rigid_right_front_wheels.stl scale=0.001 0.001 0.001
- link base_footprint: mass None -> 10
- link base_link: mass None -> 10
Joints:
- added joint drivewhl_b_l_joint: type continuous, parent base_link, child drivewhl_b_l_link, origin xyz=-0.75 0.43600000000000005 -0.425 rpy=0 0 0, axis 0 1 0
- added joint drivewhl_b_r_joint: type continuous, parent base_link, child drivewhl_b_r_link, origin xyz=-0.75 -0.43600000000000005 -0.425 rpy=0 0 0, axis 0 1 0
- added joint drivewhl_f_l_joint: type continuous, parent base_link, child drivewhl_f_l_link, origin xyz=0.75 0.43600000000000005 -0.425 rpy=0 0 0, axis 0 1 0
- added joint drivewhl_f_r_joint: type continuous, parent base_link, child drivewhl_f_r_link, origin xyz=0.75 -0.43600000000000005 -0.425 rpy=0 0 0, axis 0 1 0
- joint base_joint: child base_footprint -> base_link; parent base_link -> base_footprint
- joint lidar_joint: origin xyz=0.215 0.0 0.30 rpy=0 0 0 -> xyz=0.835 0.02 0.44 rpy=0 0 0
- joint velodyne_vlp16_joint: origin xyz=0.0 0.0 0.0 rpy=0 0 0 -> xyz=0.835 0.02 0.44 rpy=0 0 0

Commit message: Better physics

File: src/atvurdf/urdf/atvurdf_skid_steer.urdf (robot description, URDF)
Before this commit: robot atvurdf, 9 links, 8 joints
Links:
- removed link velodyne_vlp16
- added link velodyne, mass 0.125; collision cylinder length=0.0717 radius=0.0516; visual mesh filename=file://$(find atvurdf)/meshes/VLP16_base_1.dae scale=1 1 1
- link base_link: mass 10 -> 30
Joints:
- removed joint velodyne_vlp16_joint
- added joint velodyne_joint: type fixed, parent base_link, child velodyne, origin xyz=0.835 0.02 0.44 rpy=0 0 0

Commit message: Add: GPS

File: src/atvurdf/urdf/atvurdf_skid_steer.urdf (robot description, URDF)
Before this commit: robot atvurdf, 9 links, 8 joints
Links:
- added link gps_link, mass 1; collision box size=0.2 0.2 0.2; visual box size=0.2 0.2 0.2
Joints:
- added joint gps_joint: type fixed, parent base_link, child gps_link, origin xyz=0.0 0.0 0.0 rpy=0 0 0

Commit message: Physic fixes and inertia script

File: src/atvurdf/urdf/atvurdf_skid_steer.urdf (robot description, URDF)
Before this commit: robot atvurdf, 10 links, 9 joints
Links:
- link base_footprint: mass 10 -> 0.0
- link drivewhl_b_l_link: mass 10 -> 0.1
- link drivewhl_b_r_link: mass 10 -> 0.1
- link drivewhl_f_l_link: mass 10 -> 0.1
- link drivewhl_f_r_link: mass 10 -> 0.1
Joints:
- joint base_joint: child base_link -> base_footprint; parent base_footprint -> base_link

Commit message: Fixes

File: src/atvurdf/urdf/atvurdf_skid_steer.urdf (robot description, URDF)
Before this commit: robot atvurdf, 10 links, 9 joints
Joints:
- joint base_joint: origin xyz=0.0 0.0 0.0 rpy=0 0 0 -> xyz=0.0 0.0 0.772311 rpy=0 0 0
